File: Toastboard/Toastboard.sch (KiCad schematic (older format))
At the start: 44 parts

Commit message: Add values to schematic
Parts:
- removed R? (x2): R, symbol Device:R
- added C1, C2: 10u, symbol Device:C
- added D2: D_Schottky, symbol Device:D_Schottky
- added D6: LED, symbol Device:LED
- added R7: 220, symbol Device:R
- C3, C4, C5, C6: renamed from C?; value C -> 100n
- F1: renamed from F?; value Fuse -> 1A
- H1, H2, H3, H4: renamed from H?; value MountingHole_Pad -> Pad
- R1, R2, R3, R4: renamed from R?; value R -> 220
- R10, R14, R8, R9: renamed from R?; value R -> 10k
- R11, R12, R13, R15: renamed from R?; value R -> 10K
- gave numbers to parts that had none: 20
Connections:
- net +3V3: now also C2.1, D6.2 (A)
- net BTN_0: now also J1.8 (Pin_8); no longer J1.7 (Pin_7)
- net BTN_1: now also J1.9 (Pin_9); no longer J1.8 (Pin_8)
- net BTN_2: now also J1.10 (Pin_10); no longer J1.9 (Pin_9)
- net BTN_3: now also J1.11 (Pin_11); no longer J1.10 (Pin_10)
- net GND: now also J1.1 (Pin_1), C1.2, C2.2, R7.2; no longer U2.3 (OS)
- net LED_0: now also J1.4 (Pin_4); no longer J1.3 (Pin_3)
- net LED_1: now also J1.5 (Pin_5); no longer J1.4 (Pin_4)
- net LED_2: now also J1.6 (Pin_6); no longer J1.5 (Pin_5)
- net LED_3: now also J1.7 (Pin_7); no longer J1.6 (Pin_6)
- net POT_1: now also J1.16 (Pin_16); no longer J1.15 (Pin_15)
- net POT_2: now also J1.17 (Pin_17); no longer J1.16 (Pin_16)
- net SCL: now also J1.2 (Pin_2); no longer J1.1 (Pin_1)
- net SDA: now also J1.3 (Pin_3); no longer J1.2 (Pin_2)
- net SW_0: now also J1.12 (Pin_12); no longer J1.11 (Pin_11)
- net SW_1: now also J1.13 (Pin_13); no longer J1.12 (Pin_12)
- net SW_2: now also J1.14 (Pin_14); no longer J1.13 (Pin_13)
- net SW_3: now also J1.15 (Pin_15); no longer J1.14 (Pin_14)
- net +5V: now reaches J1.18 (Pin_18)
- net +5V: now also FB1.1, U3.3 (VI), C1.1
- net at J2.1 (VBUS): now also D2.2 (A); no longer F1.2
- new net: D2.1 (K), F1.2
- new net: D6.1 (K), R7.1
- no-connect marks 3 -> 4
Other:
- note added: "Buttons\n"
- note added: "DIP Switches\n"
- note added: "I2C\n"
- note added: "LEDS\n"
- note added: "Mounting Holes\n"
- note added: "Potentiometers\n"
- note added: "Power LED\n"
- note added: "ToastBoard\n"
- note added: "USB Power\n"
- moved on the sheet: C3, C4, C5, C6, D1, D3, D4, D5, F1, FB1, H1, H2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

Commit message: Initial placement
Parts:
- removed U3: AZ1117-3.3, symbol Regulator_Linear:AZ1117-3.3
- added U3: AMS1117-3.3, Package_TO_SOT_SMD:SOT-223-3_TabPin2, symbol Regulator_Linear:AMS1117-3.3
- C1, C2, C3, C4, C5, C6: footprint (none) -> Capacitor_SMD:C_0603_1608Metric_Pad1.05x0.95mm_HandSolder
- D1, D3, D4, D5, D6: footprint (none) -> LED_SMD:LED_0603_1608Metric_Pad1.05x0.95mm_HandSolder
- D2: footprint (none) -> Diode_SMD:D_0603_1608Metric_Pad1.05x0.95mm_HandSolder
- F1: footprint (none) -> Fuse:Fuse_0603_1608Metric_Pad1.05x0.95mm_HandSolder
- FB1: footprint (none) -> Inductor_SMD:L_0805_2012Metric_Pad1.15x1.40mm_HandSolder
- H1, H2, H3, H4: footprint (none) -> MountingHole:MountingHole_2.2mm_M2_DIN965_Pad
- J1: footprint (none) -> Connector_PinSocket_2.54mm:PinSocket_1x20_P2.54mm_Vertical
- J2: footprint (none) -> Connector_USB:USB_Micro-B_Amphenol_10103594-0001LF_Horizontal
- R1, R10, R11, R12, R13, R14, R15, R2, R3, R4, R5, R6, R7, R8, R9: footprint (none) -> Resistor_SMD:R_0603_1608Metric_Pad1.05x0.95mm_HandSolder
- RV1, RV2: footprint (none) -> Potentiometer_THT:Potentiometer_Vishay_248GJ-249GJ_Single_Vertical
- SW1, SW2, SW3: footprint (none) -> Button_Switch_SMD:SW_Push_1P1T_NO_6x6mm_H9.5mm
- SW4: renamed from SW5; footprint (none) -> Button_Switch_SMD:SW_Push_1P1T_NO_6x6mm_H9.5mm
- SW5: renamed from SW4; footprint (none) -> Button_Switch_SMD:SW_DIP_SPSTx04_Slide_Omron_A6S-410x_W8.9mm_P2.54mm
- U1: footprint (none) -> Package_SO:SO-8_3.9x4.9mm_P1.27mm
Connections:
- net +3V3: now also J1.18 (Pin_18), U3.2 (VO); no longer J1.20 (Pin_20)
- net +5V: now also J1.19 (Pin_19), U3.3 (VI); no longer J1.18 (Pin_18)
- net GND: now also J1.20 (Pin_20), U3.1 (GND); no longer J1.19 (Pin_19)
- net POT_1: now also J1.2 (Pin_2); no longer J1.16 (Pin_16)
- net POT_2: now also J1.3 (Pin_3); no longer J1.17 (Pin_17)
- net SCL: now also J1.16 (Pin_16); no longer J1.2 (Pin_2)
- net SDA: now also J1.17 (Pin_17); no longer J1.3 (Pin_3)
